Commit message: feat: 更新 VLA 相关功能，支持 7-DOF 机器人控制，添加夹爪支持，并完善相关文档

File: src/trossen_arm_description/urdf/generated/wxai/wxai_follower.urdf (robot description, URDF)
Before this commit: robot wxai, 23 links, 22 joints
Joints:
- removed joint left_carriage_joint
- added joint joint_6: type prismatic, parent link_6, child carriage_left, origin xyz=0.0865 0.023 0 rpy=0 0 0, axis 0 1 0, limit lower=0.0 upper=0.044 effort=400.0 velocity=0.0875
- joint right_carriage_joint: mimic joint=left_carriage_joint -> joint=joint_6
